File: power.kicad_sch (KiCad schematic)
At the start: 29 parts, among them U10 TBA1-0521E, U11 TPS72301DBV, U4 TPS7A2033PDBVR, U9 TPS7A2015PDBVR

Commit message: wip Layout
Parts:
- added C58, C59, C60, C61: 2.2u, Capacitor_SMD:C_1206_3216Metric, symbol Device:C
- added R75, R76: 1.1, Resistor_SMD:R_0603_1608Metric, symbol Device:R
- C14, C15, C19, C24, C25, C27, C48, C50: footprint Capacitor_SMD:C_0805_2012Metric -> Capacitor_SMD:C_1206_3216Metric
- C20, C29, C30: symbol Device:C_Feedthrough -> seismometer:C_Feedthrough
Connections:
- net GND: now also C20.A2 (2), C20.B2 (4), C29.A2 (2), C29.B2 (4), C30.A2 (2), C30.B2 (4), C58.2, C59.2, C60.2, C61.2; no longer C20.2, C29.2, C30.2
- net -5V: now reaches FB3.1, U10.4 (-Vout)
- net -5V: now also C59.1, R75.1
- net +5V: now reaches FB2.1, U10.6 (+Vout)
- net +5V: now also C61.1, R76.1
- new net: C58.1, R75.2
- new net: C60.1, R76.2
Other:
- moved on the sheet: C14, C27, C28, C48, C49, C50, C57, FB2, FB3, R48, R74, U4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
