File: Seismometer.kicad_sch (KiCad schematic)
At the start: 73 parts, among them U1 DLVR-F50D, U2 MC3479, U3 ADS131M04-Q1, U4 LP5907MFX-3.3, U5 Teensy4.1, X1 SIT8924BA-22-33E-8.192000G

Commit message: wip No idea? Better filters?
Parts:
- C12, C14, C15, C5, C9: MP CC0402KRX5R6BB105 -> UMK212B7105KG-T
- U3: MP ADS131M04-Q1 -> ADS131M04QPWRQ1
- U4: MP LP5907MFX-3.3 -> LP5907MFX-3.3/NOPB
Changed lines of the file:
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@@
       (effects (font (size 1.27 1.27)) hide)
     )
-    (property "MP" "LP5907MFX-3.3" (at 207.01 50.8 0)
+    (property "MP" "LP5907MFX-3.3/NOPB" (at 207.01 50.8 0)
       (effects (font (size 1.27 1.27)) hide)
     )
@@
       (effects (font (size 1.27 1.27)) hide)
     )
-    (property "MP" "CC0402KRX5R6BB105" (at 223.52 54.61 0)
+    (property "MP" "UMK212B7105KG-T" (at 223.52 54.61 0)
       (effects (font (size 1.27 1.27)) hide)
     )
@@
       (effects (font (size 1.27 1.27)) hide)
     )
-    (property "MP" "CC0402KRX5R6BB105" (at 300.99 29.21 0)
+    (property "MP" "UMK212B7105KG-T" (at 300.99 29.21 0)
       (effects (font (size 1.27 1.27)) hide)
     )
@@
       (effects (font (size 1.27 1.27)) hide)
     )
-    (property "MP" "CC0402KRX5R6BB105" (at 189.23 54.61 0)
+    (property "MP" "UMK212B7105KG-T" (at 189.23 54.61 0)
       (effects (font (size 1.27 1.27)) hide)
     )
@@
       (effects (font (size 1.27 1.27)) hide)
     )
-    (property "MP" "CC0402KRX5R6BB105" (at 87.63 53.34 0)
+    (property "MP" "UMK212B7105KG-T" (at 87.63 53.34 0)
       (effects (font (size 1.27 1.27)) hide)
     )
@@
       (effects (font (size 1.27 1.27)) hide)
     )
-    (property "MP" "CC0402KRX5R6BB105" (at 120.65 53.34 0)
+    (property "MP" "UMK212B7105KG-T" (at 120.65 53.34 0)
       (effects (font (size 1.27 1.27)) hide)
     )
@@
       (effects (font (size 1.27 1.27)) hide)
     )
-    (property "MP" "ADS131M04-Q1" (at 111.76 93.98 0)
-      (effects (font (size 1.27 1.27)) hide)
-    )
+    (property "MP" "ADS131M04QPWRQ1" (at 111.76 93.98 0)
+      (effects (font (size 1.27 1.27)) hide)
+    )
