File: geophone_input.kicad_sch (KiCad schematic)
At the start: 6 parts

Commit message: Finishing schematic
Parts:
- removed J?: Conn_01x04_Female, symbol Connector:Conn_01x04_Female
- added J4: Conn_01x03_Socket, symbol Connector:Conn_01x03_Socket
- C16: renamed from C?; footprint (none) -> Capacitor_SMD:C_0603_1608Metric_Pad1.08x0.95mm_HandSolder
- R51, R52: renamed from R?; value 10k -> 100k; footprint (none) -> Resistor_SMD:R_0603_1608Metric
- R53, R54: renamed from R?; footprint (none) -> Resistor_SMD:R_0603_1608Metric
Connections:
- net GND: now also J4.2 (Pin_2)
- net at R51.2, R53.2: now also J4.3 (Pin_3)
- net at R52.1, R54.2: now also J4.1 (Pin_1)
Other:
- moved on the sheet: C16, R51, R52, R53, R54

Commit message: Layout
Parts:
- J4: footprint (none) -> Connector_PinHeader_2.54mm:PinHeader_1x03_P2.54mm_Horizontal
Changed lines of the file:
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@@
       (effects (font (size 1.27 1.27)))
     )
-    (property "Footprint" "" (at 95.25 96.52 0)
+    (property "Footprint" "Connector_PinHeader_2.54mm:PinHeader_1x03_P2.54mm_Horizontal" (at 95.25 96.52 0)
       (effects (font (size 1.27 1.27)) hide)
     )

Commit message: Ready
Parts:
- C16: MANUFACTURER (none) -> TDK; MP (none) -> CGA3E3X7R1H224K080AB
- J4: MANUFACTURER (none) -> MOLEX; MP (none) -> 22-12-4032
- R51, R52: MANUFACTURER (none) -> VISHAY; MP (none) -> CRCW0603100KFKEA
- R53, R54: MANUFACTURER (none) -> VISHAY; MP (none) -> CRCW0603470RFKEA.
Changed lines of the file:
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@@
+      (effects (font (size 1.27 1.27)) hide)
+    )
+    (property "Description" "X7R, 16V" (at 182.88 95.25 0)
+      (effects (font (size 1.27 1.27)) hide)
+    )
+    (property "MANUFACTURER" "TDK" (at 182.88 95.25 0)
+      (effects (font (size 1.27 1.27)) hide)
+    )
+    (property "MP" "CGA3E3X7R1H224K080AB" (at 182.88 95.25 0)
       (effects (font (size 1.27 1.27)) hide)
     )
@@
       (effects (font (size 1.27 1.27)) hide)
     )
+    (property "MANUFACTURER" "VISHAY" (at 137.16 87.63 0)
+      (effects (font (size 1.27 1.27)) hide)
+    )
+    (property "MP" "CRCW0603100KFKEA" (at 137.16 87.63 0)
+      (effects (font (size 1.27 1.27)) hide)
+    )
     (pin "1")
     (pin "2")
@@
       (effects (font (size 1.27 1.27)) hide)
     )
+    (property "Description" "2.54mm right angle pin headers" (at 95.25 96.52 0)
+      (effects (font (size 1.27 1.27)) hide)
+    )
+    (property "MANUFACTURER" "MOLEX" (at 95.25 96.52 0)
+      (effects (font (size 1.27 1.27)) hide)
+    )
+    (property "MP" "22-12-4032" (at 95.25 96.52 0)
+      (effects (font (size 1.27 1.27)) hide)
+    )
     (pin "1")
     (pin "2")
@@
       (effects (font (size 1.27 1.27)) hide)
     )
+    (property "MANUFACTURER" "VISHAY" (at 137.16 104.14 0)
+      (effects (font (size 1.27 1.27)) hide)
+    )
+    (property "MP" "CRCW0603100KFKEA" (at 137.16 104.14 0)
+      (effects (font (size 1.27 1.27)) hide)
+    )
     (pin "1")
     (pin "2")
@@
     )
     (property "Datasheet" "~" (at 158.75 111.76 0)
+      (effects (font (size 1.27 1.27)) hide)
+    )
+    (property "MANUFACTURER" "VISHAY" (at 158.75 111.76 0)
+      (effects (font (size 1.27 1.27)) hide)
+    )
+    (property "MP" "CRCW0603470RFKEA." (at 158.75 111.76 0)
       (effects (font (size 1.27 1.27)) hide)
     )
@@
       (effects (font (size 1.27 1.27)) hide)
     )
+    (property "MANUFACTURER" "VISHAY" (at 158.75 80.01 0)
+      (effects (font (size 1.27 1.27)) hide)
+    )
+    (property "MP" "CRCW0603470RFKEA." (at 158.75 80.01 0)
+      (effects (font (size 1.27 1.27)) hide)
+    )

Commit message: wip No idea? Better filters?
Parts:
- R53, R54: MP CRCW0603470RFKEA. -> CRCW0603470RFKEA
Changed lines of the file:
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@@
       (effects (font (size 1.27 1.27)) hide)
     )
-    (property "MP" "CRCW0603470RFKEA." (at 158.75 111.76 0)
+    (property "MP" "CRCW0603470RFKEA" (at 158.75 111.76 0)
       (effects (font (size 1.27 1.27)) hide)
     )
@@
       (effects (font (size 1.27 1.27)) hide)
     )
-    (property "MP" "CRCW0603470RFKEA." (at 158.75 80.01 0)
+    (property "MP" "CRCW0603470RFKEA" (at 158.75 80.01 0)
       (effects (font (size 1.27 1.27)) hide)
     )
